Commit message: Migrating to RViz. Pybullet is only a physics engine and does not have build in motion planners thus causing problem while picking and placing objects.

File: models/boxes/red_box.urdf (robot description, URDF)
Before this commit: robot simple_cuboid, 1 links, 0 joints
Links:
- link base_link: mass 0.1 -> 1.0
