Commit message: Added a constraint to the keep the fingers of the robot centered at all times during simulation.
Modified the urdf gile to make the box more slender it seem more plausible to use our pybullet simulator for the simple diagonal example.

File: models/boxes/red_box (copy).urdf (robot description, URDF)
Before this commit: robot simple_cuboid, 1 links, 0 joints
Links:
- link base_link: mass 0.5 -> 1.0; geometry collision box size=0.059 0.059 0.169; collision sphere radius=1e-7
