Commit message: Committing a Work In progress arch constuction code. Added a flag to not print data in two-player-game construction. Tried building an arch manually and succeeded.

File: models/boxes/black_box_org.urdf (robot description, URDF)
Before this commit: robot simple_cuboid, 1 links, 0 joints
Links:
- link base_link: mass 0.5 -> 0.122; geometry collision box size=0.064 0.054 0.169; collision sphere radius=1e-7
